File: Multiplexer sondes.kicad_sch (KiCad schematic)
At the start: 15 parts

Commit message: Command stepper done
Parts:
- removed JP5: (no value), symbol Connector_Generic:Conn_02x02_Odd_Even
- C1: value (none) -> C; footprint (none) -> Capacitor_SMD:C_0603_1608Metric_Pad1.08x0.95mm_HandSolder
- COMMUNICATION0, POWER0, PWML0: value (none) -> FH254-108DF08500V; footprint (none) -> Connector_PinHeader_2.54mm:PinHeader_1x08_P2.54mm_Vertical
- H0, H1, H2, H3: value (none) -> MountingHole_Pad; footprint (none) -> MountingHole:MountingHole_3.2mm_M3
- ICSP1: value (none) -> ICSP; footprint (none) -> Connector_PinSocket_2.54mm:PinSocket_2x03_P2.54mm_Vertical
- J1: value (none) -> OIP; footprint (none) -> Connector_Coaxial:SMA_Molex_73251-1153_EdgeMount_Horizontal
- J2: value (none) -> DB9_Female_MountingHoles; footprint (none) -> Connector_Dsub:DSUB-9_Female_Horizontal_P2.77x2.84mm_EdgePinOffset4.94mm_Housed_MountingHolesOffset7.48mm
- JP6: value (none) -> FH254-110DF08500V; footprint (none) -> Connector_PinHeader_2.54mm:PinHeader_1x10_P2.54mm_Vertical
- R1: value (none) -> R; footprint (none) -> Resistor_SMD:R_0603_1608Metric_Pad0.98x0.95mm_HandSolder
- XIO0: value (none) -> 18x2F-H8.5; footprint (none) -> Connector_PinHeader_2.54mm:PinHeader_2x18_P2.54mm_Vertical
Connections:
- no-connect marks 10 -> 62
Other:
- moved on the sheet: H0, H1, H2, H3
