File: Relais.kicad_sch (KiCad schematic)
At the start: 16 parts

Commit message: Command stepper done
Parts:
- K1, K10, K11, K12, K13, K14, K15, K16, K2, K3, K4, K5, K6, K7, K8, K9: value (none) -> 3570-1411-053; footprint (none) -> Relay_THT:Relay_SPST_StandexMeder_MS_Form1AB
Connections:
- net GND: now also K8.5
